Commit message: addded force/torque sensor

File: models/kopterworx/urdf/kopterworx.urdf.xacro (robot description, xacro)
@@ -139,3 +139,4 @@
     <origin xyz="0.25 0 -0.1" rpy="0 0 0"/>
   </xacro:gimbal_macro> -->
+<!--Adding force/torque sensor to the base_link of a kopterworx-->
 </robot>

File: models/kopterworx/urdf/multirotor_base.urdf.xacro (robot description, xacro)
@@ -80,59 +80,4 @@
       <limit upper="0" lower="0" effort="0" velocity="0" />
     </joint>
-    <!--Adding a sensor link and joint and a sensor plugin-->
-      <joint name="sensor_joint" type="revolute">
-        <parent link="${robot_namespace}/base_link"/>
-        <child link="sensor_link"/>
-        <limit upper="100" lower="-100" effort="100" velocity="100" />
-        <axis xyz="0 0 1" />
-      </joint>
-      <link name="sensor_link">
-      <visual>
-        <origin xyz="0 0 0" rpy="0 0 0"/>
-        <geometry>
-          <cylinder length="0.1" radius="0.02"/>
-        </geometry>
-        <material name="red">
-          <color rgba="1 0 0 1"/>
-        </material>
-      </visual>
-      <collision>
-        <origin xyz="0 0 0" rpy="0 0 0"/>
-        <geometry>
-          <box size="0.1 0.1 0.1"/>
-        </geometry>
-      </collision>
-      <inertial>
-        <origin xyz="0 0 0" rpy="0 0 0"/>
-        <mass value="0.1"/>
-        <inertia ixx="0.001" ixy="0.0" ixz="0.0" iyy="0.001" iyz="0.0" izz="0.001"/>
-      </inertial>
-      </link>
-      <gazebo reference="sensor_link">
-        <provideFeedback>true</provideFeedback>
-      </gazebo>
-      <gazebo reference="sensor_joint">
-        <provideFeedback>true</provideFeedback>
-      </gazebo>
-      <gazebo reference="${robot_namespace}/base_link">
-        <provideFeedback>true</provideFeedback>
-      </gazebo>
-      <gazebo>
-        <plugin name="ft_sensor" filename="libgazebo_ros_ft_sensor.so">
-          <!--<updateRate>100.0</updateRate>-->
-          <updateRate>100.0</updateRate>
-          <topicName>/${robot_namespace}/ft_sensor</topicName>
-          <jointName>sensor_joint</jointName>
-        </plugin>
-        <provideFeedback>true</provideFeedback>
-      </gazebo>
-      <!--
-      <gazebo>
-        <plugin name="ft_sensor" filename="libgazebo_ros_ft_sensor.so">
-          <updateRate>100.0</updateRate>
-          <topic>/${robot_namespace}/ft_sensor</topic>
-          <jointName>${robot_namespace}/sensor_joint</jointName>
-        </plugin>
-      </gazebo>-->
     <!-- attach multirotor_base_plugin to the base_link -->
     <gazebo>
@@ -143,4 +88,30 @@
       </plugin>
     </gazebo>
+  <!--tu je bio </xacro:macro> prije -->
+  <!--force/torque sensor link and joint-->
+    <link name="sensor_link">
+    <visual>
+      <origin xyz="0 0 0" rpy="0 0 0"/>
+      <geometry>
+        <box size="0.1 0.1 0.1"/>
+      </geometry>
+    </visual>
+    <collision>
+      <origin xyz="0 0 0" rpy="0 0 0"/>
+      <geometry>
+        <box size="0.1 0.1 0.1"/>
+      </geometry>
+    </collision>
+    <inertial>
+      <origin xyz="0 0 0" rpy="0 0 0"/>
+      <mass value="0.1"/>
+      <inertia ixx="0.001" ixy="0.0" ixz="0.0" iyy="0.001" iyz="0.0" izz="0.001"/>
+    </inertial>
+    </link>
+    <joint name="sensor_joint" type="fixed">
+      <parent link="${robot_namespace}/base_link"/>
+      <child link="sensor_link"/>
+      <origin xyz="0 0 0" rpy="0 0 0"/>
+    </joint>
   </xacro:macro>
   <!-- Rotor joint and link -->
